File: FFaE/pow.kicad_sch (KiCad schematic)
At the start: 9 parts, among them U3 L7805, U4 L7809

Commit message: Dump
Parts:
- renumbered C22 to C21, C20 to C22, D6 to D3, D3 to D4, D4 to D6
Other:
- moved on the sheet: C21, C22, C23, D3, D4, D5, D6, U3, U4
