File: FFaE/FFaE.kicad_sch (KiCad schematic)
At the start: 0 parts

Commit message: Dump
Parts:
- added J1: Conn_01x02_Pin, Connector_Phoenix_MSTB:PhoenixContact_MSTBVA_2,5_2-G_1x02_P5.00mm_Vertical, symbol Connector:Conn_01x02_Pin
- added J10, J11: Barrel_Jack, symbol Connector:Barrel_Jack
- added J2: FUZZ_OUTPUT, TestPoint:TestPoint_THTPad_D2.0mm_Drill1.0mm, symbol Connector_Generic:Conn_01x01
- added J3: ECHO_OUTPUT, TestPoint:TestPoint_THTPad_D2.0mm_Drill1.0mm, symbol Connector_Generic:Conn_01x01
- added J4: FUZZ_INPUT, TestPoint:TestPoint_THTPad_D2.0mm_Drill1.0mm, symbol Connector_Generic:Conn_01x01
- added J5: ECHO_INPUT, TestPoint:TestPoint_THTPad_D2.0mm_Drill1.0mm, symbol Connector_Generic:Conn_01x01
- added J6: INPUT, TestPoint:TestPoint_THTPad_D2.0mm_Drill1.0mm, symbol Connector_Generic:Conn_01x01
- added J7: OUTPUT, TestPoint:TestPoint_THTPad_D2.0mm_Drill1.0mm, symbol Connector_Generic:Conn_01x01
- added J8: INPUT_GND, TestPoint:TestPoint_THTPad_D2.0mm_Drill1.0mm, symbol Connector_Generic:Conn_01x01
- added J9: OUTPUT_GND, TestPoint:TestPoint_THTPad_D2.0mm_Drill1.0mm, symbol Connector_Generic:Conn_01x01
- added SW1, SW2, SW3, SW4, SW5, SW6: SW_SPDT, symbol Switch:SW_SPDT
Connections:
- net Power management/POW+: now also J1.1 (Pin_1)
- net Power management/POW-: now also J1.2 (Pin_2)
- new net: J10.1, SW5.2 (B)
- new net: J10.2, SW6.2 (B)
- new net: J11.1, SW5.3 (C)
- new net: J11.2, SW6.1 (A)
- new net GND: J8.1 (Pin_1), J9.1 (Pin_1)
- new net echo_input: J5.1 (Pin_1), SW1.3 (C), SW3.1 (A)
- new net echo_output: J3.1 (Pin_1), SW2.2 (B)
- new net fuzz_input: J4.1 (Pin_1), SW2.1 (A), SW3.3 (C)
- new net fuzz_output: J2.1 (Pin_1), SW1.2 (B)
- new net input: J6.1 (Pin_1), SW3.2 (B)
- new net output: J7.1 (Pin_1), SW1.1 (A), SW2.3 (C)
Other:
- added sheet Input buffer 1 (buffer.kicad_sch)
- added sheet Input buffer 2 (buffer.kicad_sch)

Commit message: PCB v0
Parts:
- removed J1: Conn_01x02_Pin, Connector_Phoenix_MSTB:PhoenixContact_MSTBVA_2,5_2-G_1x02_P5.00mm_Vertical, symbol Connector:Conn_01x02_Pin
- removed J2: FUZZ_OUTPUT, TestPoint:TestPoint_THTPad_D2.0mm_Drill1.0mm, symbol Connector_Generic:Conn_01x01
- removed J3: ECHO_OUTPUT, TestPoint:TestPoint_THTPad_D2.0mm_Drill1.0mm, symbol Connector_Generic:Conn_01x01
- removed J4: FUZZ_INPUT, TestPoint:TestPoint_THTPad_D2.0mm_Drill1.0mm, symbol Connector_Generic:Conn_01x01
- removed J5: ECHO_INPUT, TestPoint:TestPoint_THTPad_D2.0mm_Drill1.0mm, symbol Connector_Generic:Conn_01x01
- removed J6: INPUT, TestPoint:TestPoint_THTPad_D2.0mm_Drill1.0mm, symbol Connector_Generic:Conn_01x01
- removed J7: OUTPUT, TestPoint:TestPoint_THTPad_D2.0mm_Drill1.0mm, symbol Connector_Generic:Conn_01x01
- removed J8: INPUT_GND, TestPoint:TestPoint_THTPad_D2.0mm_Drill1.0mm, symbol Connector_Generic:Conn_01x01
- removed J9: OUTPUT_GND, TestPoint:TestPoint_THTPad_D2.0mm_Drill1.0mm, symbol Connector_Generic:Conn_01x01
- removed SW1, SW2, SW3, SW4, SW5, SW6: SW_SPDT, symbol Switch:SW_SPDT
- added D10, D11, D12: LED, Connector_JST:JST_PH_B2B-PH-K_1x02_P2.00mm_Vertical, symbol Device:LED
- added D8, D9: 1N4007, Diode_THT:D_DO-41_SOD81_P10.16mm_Horizontal, symbol Diode:1N4007
- added J1: DC_in, Connector_JST:JST_PH_B2B-PH-K_1x02_P2.00mm_Vertical, symbol Connector_Generic:Conn_01x02
- added JP1, JP2, JP3, JP4, JP5, JP6: SolderJumper_2_Open, Jumper:SolderJumper-2_P1.3mm_Open_RoundedPad1.0x1.5mm, symbol Jumper:SolderJumper_2_Open
- added R24, R25: 220R, Resistor_THT:R_Axial_DIN0207_L6.3mm_D2.5mm_P7.62mm_Horizontal, symbol Device:R
- added SW1: Shoegaze, Connector_JST:JST_PH_B2B-PH-K_1x02_P2.00mm_Vertical, symbol Switch:SW_DPDT_x2
- added U7, U8: UB2-5NUN, KiCAD_lib:UB2-5NUN, symbol KiCAD__lib:UB2-5NUN
- J10: value Barrel_Jack -> Input_Jack; footprint (none) -> Connector_JST:JST_PH_B2B-PH-K_1x02_P2.00mm_Vertical
- J11: value Barrel_Jack -> Output_Jack; footprint (none) -> Connector_JST:JST_PH_B2B-PH-K_1x02_P2.00mm_Vertical
Connections:
- net GND: now also J10.2, J11.2, D8.2 (A), D9.2 (A), R24.2, R25.1, U7.8, U8.8
- net Power management/POW+: now also J1.1 (Pin_1)
- net Power management/POW-: now also J1.2 (Pin_2)
- net at J10.1: now also JP1.1 (A), JP2.1 (A)
- net at J11.1: now also JP3.2 (B), JP4.2 (B)
- new net: D10.1 (K), R25.2
- new net: D8.1 (K), D9.1 (K), SW1.1 (A), U7.1, U8.1
- new net: D11.1 (K), U7.7
- new net: D12.1 (K), U7.5
- new net: R24.1, U7.6
- new net +5V: D10.2 (A), D11.2 (A), D12.2 (A), SW1.2 (B)
- new net Echo_input: U7.4, U8.2
- new net Echo_output: U8.6
- new net Fuzz_input: U7.2, U8.5
- new net Fuzz_output: U8.3
- new net Input: JP2.2 (B), JP5.2 (B), U7.3
- new net Input Buffer/Input: JP1.2 (B)
- new net Input Buffer/Output: JP5.1 (A)
- new net Output: JP4.1 (A), JP6.1 (A), U8.4, U8.7
- new net Output Buffer/Input: JP6.2 (B)
- new net Output Buffer/Output: JP3.1 (A)
- no-connect marks 0 -> 1
Other:
- sheet Input buffer 1 renamed Input Buffer
- sheet Input buffer 2 renamed Output Buffer
- moved on the sheet: J11
