File: FFaE/buffer.kicad_sch (KiCad schematic)
At the start: 2 parts, among them U5 LM741

Commit message: PCB v0
Parts:
- added R20, R22: 100k, Resistor_THT:R_Axial_DIN0207_L6.3mm_D2.5mm_P7.62mm_Horizontal, symbol Device:R
Connections:
- net +9V: now also R20.1
- net GND: now also R22.2
- net Input: now also R20.2, R22.1
Other:
- moved on the sheet: C24
