File: FFaE/echo.kicad_sch (KiCad schematic)
At the start: 30 parts, among them U2 PT2399

Commit message: Dump
Parts:
- added C26: 100nF, Capacitor_THT:C_Rect_L4.0mm_W2.5mm_P2.50mm, symbol Device:C
- added D7: 1N4148, Diode_THT:D_DO-35_SOD27_P7.62mm_Horizontal, symbol Diode:1N4148
- added Q1: BC337, Package_TO_SOT_THT:TO-92_Inline, symbol Transistor_BJT:BC337
- added R19: 100k, Resistor_THT:R_Axial_DIN0207_L6.3mm_D2.5mm_P7.62mm_Horizontal, symbol Device:R
- renumbered C9 to C10, C10 to C11, C11 to C12, C12 to C13, C13 to C14, C14 to C15, C15 to C16, C16 to C17, C17 to C18, C18 to C19, C19 to C20, C4 to C5, C5 to C6, C6 to C7, C7 to C8, C8 to C9
Connections:
- net +5V: now also D7.1 (K), R19.2
- net GND: now also C26.2, Q1.3 (E)
- net at R8.2, U2.6 (VCO): now also Q1.1 (C)
- new net: C26.1, D7.2 (A), Q1.2 (B), R19.1
- no-connect marks 1 -> 3
Other:
- note added: "Short GND and AGND Brigde pin 3 and 4"
- moved on the sheet: C7, C9

Commit message: PCB v0
Parts:
- RV2: footprint Potentiometer_THT:Potentiometer_Vishay_148-149_Single_Horizontal -> Connector_JST:JST_PH_B2B-PH-K_1x02_P2.00mm_Vertical
- RV3: footprint Potentiometer_THT:Potentiometer_Vishay_148-149_Single_Horizontal -> Connector_JST:JST_PH_B3B-PH-K_1x03_P2.00mm_Vertical
Connections:
- net at RV2.1: now also R8.1
- net at RV2.3: no longer R8.1
Other:
- moved on the sheet: RV2
Changed lines of the file:
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@@
 			)
 		)
-		(property "Footprint" "Potentiometer_THT:Potentiometer_Vishay_148-149_Single_Horizontal"
+		(property "Footprint" "Connector_JST:JST_PH_B3B-PH-K_1x03_P2.00mm_Vertical"
 			(at 207.01 90.17 0)
 			(effects
@@
 	(symbol
 		(lib_id "Device:R_Potentiometer")
-		(at 73.66 101.6 90)
-		(unit 1)
-		(exclude_from_sim no)
-		(in_bom yes)
-		(on_board yes)
-		(dnp no)
-		(fields_autoplaced yes)
+		(at 73.66 101.6 270)
+		(mirror x)
+		(unit 1)
+		(exclude_from_sim no)
+		(in_bom yes)
+		(on_board yes)
+		(dnp no)
 		(property "Reference" "RV2"
 			(at 73.66 105.41 90)
@@
 			)
 		)
-		(property "Footprint" "Potentiometer_THT:Potentiometer_Vishay_148-149_Single_Horizontal"
+		(property "Footprint" "Connector_JST:JST_PH_B2B-PH-K_1x02_P2.00mm_Vertical"
 			(at 73.66 101.6 0)
 			(effects
