File: FFaE/fuzz.kicad_sch (KiCad schematic)
At the start: 14 parts, among them U1 LM741

Commit message: Dump
Parts:
- added C3: 100nF, Capacitor_THT:C_Rect_L4.0mm_W2.5mm_P2.50mm, symbol Device:C
- renumbered C3 to C4, R5 to R1, R1 to R4, R4 to R5
Connections:
- net +9V: now also C3.2
- net GND: now also C3.1
Changed lines of the file:
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@@
 (kicad_sch
-	(version 20231120)
+	(version 20250114)
 	(generator "eeschema")
-	(generator_version "8.0")
+	(generator_version "9.0")
 	(paper "A4")
 	(junction
@@
 	)
 	(junction
+		(at 130.81 66.04)
+		(diameter 0)
+		(color 0 0 0 0)
+	)
+	(junction
 		(at 151.13 66.04)
 		(diameter 0)
@@
 	(wire
 		(pts
+			(xy 123.19 68.58) (xy 123.19 66.04)
+		)
+		(stroke
+			(width 0)
+			(type default)
+		)
+	)
+	(wire
+		(pts
 			(xy 130.81 90.17) (xy 130.81 133.35)
 		)
@@
 		(shape input)
 		(at 90.17 80.01 180)
-		(fields_autoplaced yes)
 		(effects
 			(font
@@
 		(shape output)
 		(at 231.14 82.55 0)
-		(fields_autoplaced yes)
 		(effects
 			(font
@@
 		(dnp no)
 		(fields_autoplaced yes)
-		(property "Reference" "R4"
+		(property "Reference" "R5"
 			(at 184.15 123.1899 0)
 			(effects
@@
 			(project "FFaE"
 				(path "/aa3b89a1-f9e5-4532-935a-0db76e43367b/e1933313-1d6e-4a08-82a1-b82dd98874aa"
-					(reference "R4")
+					(reference "R5")
 					(unit 1)
 				)
@@
 		)
 		(instances
-			(project ""
+			(project "FFaE"
 				(path "/aa3b89a1-f9e5-4532-935a-0db76e43367b/e1933313-1d6e-4a08-82a1-b82dd98874aa"
 					(reference "D1")
@@
 		)
 		(instances
-			(project ""
+			(project "FFaE"
 				(path "/aa3b89a1-f9e5-4532-935a-0db76e43367b/e1933313-1d6e-4a08-82a1-b82dd98874aa"
 					(reference "U1")
+					(unit 1)
+				)
+			)
+		)
+	)
+	(symbol
+		(lib_id "power:Earth")
+		(at 123.19 68.58 0)
+		(unit 1)
+		(exclude_from_sim no)
+		(in_bom yes)
+		(on_board yes)
+		(dnp no)
+		(fields_autoplaced yes)
+		(property "Reference" "#PWR01"
+			(at 123.19 74.93 0)
+			(effects
+				(font
+					(size 1.27 1.27)
+				)
+				(hide yes)
+			)
+		)
+		(property "Value" "GND"
+			(at 123.19 73.66 0)
+			(effects
+				(font
+					(size 1.27 1.27)
+				)
+			)
+		)
+		(property "Footprint" ""
+			(at 123.19 68.58 0)
+			(effects
+				(font
+					(size 1.27 1.27)
+				)
+				(hide yes)
+			)
+		)
+		(property "Datasheet" "~"
+			(at 123.19 68.58 0)
+			(effects
+				(font
+					(size 1.27 1.27)
+				)
+				(hide yes)
+			)
+		)
+		(property "Description" "Power symbol creates a global label with name \"Earth\""
+			(at 123.19 68.58 0)
+			(effects
+				(font
+					(size 1.27 1.27)
+				)
+				(hide yes)
+			)
+		)
+		(pin "1"
+		)
+		(instances
+			(project "FFaE"
+				(path "/aa3b89a1-f9e5-4532-935a-0db76e43367b/e1933313-1d6e-4a08-82a1-b82dd98874aa"
+					(reference "#PWR01")
+					(unit 1)
+				)
+			)
+		)
+	)
+	(symbol
+		(lib_id "Device:C")
+		(at 127 66.04 90)
+		(unit 1)
+		(exclude_from_sim no)
+		(in_bom yes)
+		(on_board yes)
+		(dnp no)
+		(fields_autoplaced yes)
+		(property "Reference" "C3"
+			(at 127 58.42 90)
+			(effects
+				(font
+					(size 1.27 1.27)
+				)
+			)
+		)
+		(property "Value" "100nF"
+			(at 127 60.96 90)
+			(effects
+				(font
+					(size 1.27 1.27)
+				)
+			)
+		)
+		(property "Footprint" "Capacitor_THT:C_Rect_L4.0mm_W2.5mm_P2.50mm"
+			(at 130.81 65.0748 0)
+			(effects
+				(font
+					(size 1.27 1.27)
+				)
+				(hide yes)
+			)
+		)
+		(property "Datasheet" "~"
+			(at 127 66.04 0)
+			(effects
+				(font
+					(size 1.27 1.27)
+				)
+				(hide yes)
+			)
+		)
+		(property "Description" "Unpolarized capacitor"
+			(at 127 66.04 0)
+			(effects
+				(font
+					(size 1.27 1.27)
+				)
+				(hide yes)
+			)
+		)
+		(pin "1"
+		)
+		(pin "2"
+		)
+		(instances
+			(project "FFaE"
+				(path "/aa3b89a1-f9e5-4532-935a-0db76e43367b/e1933313-1d6e-4a08-82a1-b82dd98874aa"
+					(reference "C3")
 					(unit 1)
 				)
@@
 		(dnp no)
 		(fields_autoplaced yes)
-		(property "Reference" "R5"
+		(property "Reference" "R1"
 			(at 111.76 87.6299 0)
 			(effects
@@
 			(project "FFaE"
 				(path "/aa3b89a1-f9e5-4532-935a-0db76e43367b/e1933313-1d6e-4a08-82a1-b82dd98874aa"
-					(reference "R5")
+					(reference "R1")
 					(unit 1)
 				)
@@
 		(dnp no)
 		(fields_autoplaced yes)
-		(property "Reference" "#PWR010"
+		(property "Reference" "#PWR02"
 			(at 151.13 67.31 0)
 			(effects
@@
 		)
 		(instances
-			(project ""
+			(project "FFaE"
 				(path "/aa3b89a1-f9e5-4532-935a-0db76e43367b/e1933313-1d6e-4a08-82a1-b82dd98874aa"
-					(reference "#PWR010")
+					(reference "#PWR02")
 					(unit 1)
 				)
@@
 		(dnp no)
 		(fields_autoplaced yes)
-		(property "Reference" "#PWR09"
+		(property "Reference" "#PWR03"
 			(at 151.13 142.24 0)
 			(effects
@@
 			(project "FFaE"
 				(path "/aa3b89a1-f9e5-4532-935a-0db76e43367b/e1933313-1d6e-4a08-82a1-b82dd98874aa"
-					(reference "#PWR09")
+					(reference "#PWR03")
 					(unit 1)
 				)
@@
 		)
 		(instances
-			(project ""
+			(project "FFaE"
 				(path "/aa3b89a1-f9e5-4532-935a-0db76e43367b/e1933313-1d6e-4a08-82a1-b82dd98874aa"
 					(reference "D2")
@@
 		(dnp no)
 		(fields_autoplaced yes)
-		(property "Reference" "R1"
+		(property "Reference" "R4"
 			(at 184.15 87.6299 0)
 			(effects
@@
 			(project "FFaE"
 				(path "/aa3b89a1-f9e5-4532-935a-0db76e43367b/e1933313-1d6e-4a08-82a1-b82dd98874aa"
-					(reference "R1")
+					(reference "R4")
 					(unit 1)
 				)
@@
 		(dnp no)
 		(fields_autoplaced yes)
-		(property "Reference" "C3"
+		(property "Reference" "C4"
 			(at 219.71 74.93 90)
 			(effects
@@
 			(project "FFaE"
 				(path "/aa3b89a1-f9e5-4532-935a-0db76e43367b/e1933313-1d6e-4a08-82a1-b82dd98874aa"
-					(reference "C3")
+					(reference "C4")
 					(unit 1)
 				)

Commit message: PCB v0
Parts:
- RV1: footprint Potentiometer_THT:Potentiometer_Vishay_148-149_Single_Horizontal -> Connector_JST:JST_PH_B2B-PH-K_1x02_P2.00mm_Vertical
Connections:
- net at D1.2 (A), D2.1 (K): now also RV1.1; no longer RV1.3
Changed lines of the file:
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@@
 		(lib_id "Device:R_Potentiometer")
 		(at 149.86 93.98 0)
+		(mirror x)
 		(unit 1)
 		(exclude_from_sim no)
@@
 		(on_board yes)
 		(dnp no)
-		(fields_autoplaced yes)
 		(property "Reference" "RV1"
-			(at 147.32 92.7099 0)
+			(at 147.32 95.2501 0)
 			(effects
 				(font
@@
 		)
 		(property "Value" "B50K"
-			(at 147.32 95.2499 0)
+			(at 147.32 92.7101 0)
 			(effects
 				(font
@@
 			)
 		)
-		(property "Footprint" "Potentiometer_THT:Potentiometer_Vishay_148-149_Single_Horizontal"
+		(property "Footprint" "Connector_JST:JST_PH_B2B-PH-K_1x02_P2.00mm_Vertical"
 			(at 149.86 93.98 0)
 			(effects
